File: FrostByte_IRCamera_PCB.kicad_pcb (KiCad board)
At the start: 4 copper layers, 91 x 62 mm, 85 parts, among them IC1 USB6B1RL, J1 Power_Input, J2 Conn_01x02_Socket, J3 Conn_01x04_Socket, J4 Conn_02x10, J5 UART, J6 USB4120-03-C_REVA6, Q1 SI3127DV-T1-GE3, SW1 SW_Push, SW2 SW_Push, U1 AP63203WU-7, U2 ESP32-S3-WROOM-1, U3 SN74AXC4T245PWR, U4 TCA9517DGKR, Y1 32.768kHz

Commit message: Rev A PCB Ordered
Parts:
- removed the G*** at (152.0, 121.0)
- removed IC1: USB6B1RL, footprints:SOIC127P600X175-8N
- removed TP11: TestPoint, TestPoint:TestPoint_THTPad_1.5x1.5mm_Drill0.7mm
- added C19: 1uF, Capacitor_SMD:C_0805_2012Metric_Pad1.18x1.45mm_HandSolder, F.Cu at (110.6, 113.4)
- added G***: LOGO, footprints:rinkstat_logo, F.Cu at (178.7, 101.4)
- added R25: 10k, Resistor_SMD:R_0805_2012Metric_Pad1.20x1.40mm_HandSolder, F.Cu at (127.0, 107.8)
- added R26: 47k, Resistor_SMD:R_0805_2012Metric_Pad1.20x1.40mm_HandSolder, F.Cu at (130.1, 116.4)
- added R27: 47k, Resistor_SMD:R_0805_2012Metric_Pad1.20x1.40mm_HandSolder, F.Cu at (126.7, 111.9)
- added R28: 10k, Resistor_SMD:R_0805_2012Metric_Pad1.20x1.40mm_HandSolder, F.Cu at (138.9, 104.4)
- added U5: USB6B1RL, footprints:SOIC127P600X175-8N, F.Cu at (116.2, 86.4)
- moved 3v3 93.9 mm to (118.2, 115.4)
- moved 2v8 91.9 mm to (114.7, 115.4)
- moved C3 44.0 mm to (158.7, 107.2), turned to 0 degrees
- moved C2 40.5 mm to (152.5, 115.7), turned to 0 degrees
- moved U1 39.4 mm to (155.7, 111.7), turned to 0 degrees
- moved C1 39.2 mm to (154.8, 123.2)
- moved R20 36.7 mm to (115.6, 95.2), turned to -90 degrees
- moved FB1 34.3 mm to (162.2, 123.9)
- moved R17 34.3 mm to (165.9, 96.1)
- moved F2 34.1 mm to (165.4, 103.1)
- moved D1 32.9 mm to (170.6, 130.2)
- moved H3 32.9 mm to (104.6, 128.2)
- moved H4 32.9 mm to (183.6, 128.2)
- moved J6 32.9 mm to (117.3, 76.8)
- moved SCL 32.9 mm to (111.1, 131.2)
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- renumbered TP6 to 2v8, TP1 to 3v3, TP4 to CLK, TP2 to CS, TP5 to MISO, TP3 to MOSI, TP10 to RX, TP8 to SCL, TP7 to SDA, TP9 to TX
Connections:
- C17 pad 1: +2V8 -> +3.3V
- C18 pad 1: +3.3V -> GND
- C18 pad 2: GND -> +2V8
- R20 pad 1: /MCU/SDA_B -> +2V8
- R20 pad 2: +2V8 -> /MCU/SCL_B
- R21 pad 2: /MCU/SCL_B -> /MCU/SDA_B
- U4 pad 1: +3.3V -> +2V8
- U4 pad 2: /MCU/SCL_A -> /MCU/SCL_B
- U4 pad 3: /MCU/SDA_A -> /MCU/SDA_B
- U4 pad 6: /MCU/SDA_B -> /MCU/SDA_A
- U4 pad 7: /MCU/SCL_B -> /MCU/SCL_A
- U4 pad 8: +2V8 -> +3.3V
Routing:
- net /MCU/VSYNC: track 0.00 -> 97.8 mm, vias 0 -> 1
- net +5V: track 20.3 -> 115.6 mm, vias 0 -> 3
- net /MCU/CAM_TEMP: track 11.9 -> 60.0 mm, vias 0 -> 2
- net /MCU/SPI_CS: track 26.8 -> 65.5 mm
- net /MCU/SPI_MISO: track 47.6 -> 86.2 mm
- net /MCU/EN_SPI: track 16.7 -> 53.8 mm, vias 0 -> 2
- net /MCU/SPI_MOSI: track 31.0 -> 65.9 mm
- net /MCU/SPI_CLK: track 32.3 -> 65.0 mm
- net /Power_Circuitry/source: track 52.8 -> 30.7 mm
- net +2V8: track 19.7 -> 36.3 mm, vias 6 -> 8
- net Net-(U1-SW): track 15.6 -> 0.00 mm
- net /MCU/SCL_A: track 59.0 -> 69.8 mm
- net +3.3V: track 48.0 -> 57.9 mm
- net Net-(FB1-Pad1): track 3.81 -> 13.4 mm
- net /MCU/SDA_A: track 59.1 -> 68.3 mm
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- added copper zone on F.Cu, net +3.3V
- added copper zone on F.Cu, net /Power_Circuitry/source
- added copper zone on F.Cu, net GND
- added copper zone on F.Cu, net Net-(U1-EN)
- added copper zone on F.Cu, net Net-(U1-SW)
- removed copper zone on In2.Cu, net +5V
Other:
- board text added: "DNP"
